File: boards/arduino-shield-xyz-stepper.brd (EAGLE design)
At the start: 76.2 x 55.5 mm, 8 parts, among them IC1 2967-MP6500, IC2 2967-MP6500, IC3 2967-MP6500, J4 ARDUINO_R3_SHIELD

Commit message: xyz stepper control
Parts:
- added J5: (no value), SparkFun-Connectors:1X09
Connections:
- new net N$16: J4.D12, J5.2
- new net N$17: J4.D11, J5.3
- new net N$18: J4.D10, J5.4
- new net N$19: J4.D9, J5.5
- new net N$22: J4.D8, J5.6
- new net N$23: J4.D7, J5.7
- new net N$24: J4.D6, J5.8
- new net N$25: J4.D5, J5.9
- net GND: now also J5.1
Routing:
- net N$25: track 0.00 -> 4.59 mm
- net N$24: track 0.00 -> 4.59 mm
- net N$23: track 0.00 -> 4.59 mm
- net N$22: track 0.00 -> 4.06 mm
- net N$19: track 0.00 -> 4.06 mm
- net N$18: track 0.00 -> 4.06 mm
- net N$17: track 0.00 -> 4.06 mm
- net N$16: track 0.00 -> 4.06 mm
- net EN2: track 55.0 -> 56.9 mm
- net STEP2: track 38.5 -> 40.0 mm
Changed lines of the file:
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@@
 <text x="13.208" y="42.418" size="1.016" layer="21">DIR3</text>
 <text x="20.828" y="46.482" size="1.016" layer="21" rot="R180">EN3</text>
-<text x="16.002" y="7.112" size="1.016" layer="21" rot="R45">EN2</text>
-<text x="11.43" y="7.62" size="1.016" layer="21" rot="R45">STEP2</text>
-<text x="6.858" y="7.62" size="1.016" layer="21" rot="R45">DIR2</text>
+<text x="14.478" y="7.112" size="1.016" layer="21" rot="R45">EN2</text>
+<text x="10.922" y="6.604" size="1.016" layer="21" rot="R45">STEP2</text>
+<text x="6.858" y="7.112" size="1.016" layer="21" rot="R45">DIR2</text>
 <text x="42.164" y="54.61" size="1.27" layer="21" rot="R180">trashrobot5-arduino-xyz-stepper november 2020</text>
+<text x="40.64" y="9.398" size="1.27" layer="21" rot="R180">GND</text>
 </plain>
 <attributes>
@@
 </element>
 <element name="J4" library="SparkFun-Boards" package="UNO_R3_SHIELD" value="ARDUINO_R3_SHIELD" x="56.896" y="0" rot="R90"/>
+<element name="J5" library="SparkFun-Connectors" package="1X09" value="" x="36.576" y="6.604" rot="R180"/>
 </elements>
 <signals>
@@
 <contactref element="J4" pad="GND@0"/>
 <contactref element="J4" pad="GND@2"/>
+<contactref element="J5" pad="1"/>
 </signal>
 <signal name="N$30">
@@
 <contactref element="IC3" pad="1"/>
 <contactref element="J4" pad="D4"/>
-<wire x1="12.446" y1="2.54" x2="18.034" y2="8.128" width="0.4064" layer="1"/>
-<wire x1="18.034" y1="8.128" x2="29.972" y2="8.128" width="0.4064" layer="1"/>
-<wire x1="29.972" y1="8.128" x2="29.972" y2="34.036" width="0.4064" layer="1"/>
+<wire x1="29.972" y1="9.144" x2="29.972" y2="34.036" width="0.4064" layer="1"/>
 <wire x1="29.972" y1="34.036" x2="27.94" y2="36.068" width="0.4064" layer="1"/>
 <wire x1="27.94" y1="36.068" x2="21.59" y2="36.068" width="0.4064" layer="1"/>
+<wire x1="12.446" y1="2.54" x2="12.446" y2="6.858" width="0.4064" layer="1"/>
+<wire x1="12.446" y1="6.858" x2="14.732" y2="9.144" width="0.4064" layer="1"/>
+<wire x1="14.732" y1="9.144" x2="29.972" y2="9.144" width="0.4064" layer="1"/>
 </signal>
 <signal name="N$5">
@@
 <contactref element="J4" pad="D3"/>
 <wire x1="9.906" y1="2.54" x2="10.16" y2="2.794" width="0.4064" layer="1"/>
-<wire x1="10.16" y1="2.794" x2="10.16" y2="5.08" width="0.4064" layer="1"/>
-<wire x1="10.16" y1="5.08" x2="15.24" y2="10.16" width="0.4064" layer="1"/>
-<wire x1="15.24" y1="10.16" x2="28.448" y2="10.16" width="0.4064" layer="1"/>
+<wire x1="10.16" y1="2.794" x2="10.16" y2="7.62" width="0.4064" layer="1"/>
+<wire x1="10.16" y1="7.62" x2="12.7" y2="10.16" width="0.4064" layer="1"/>
+<wire x1="12.7" y1="10.16" x2="28.448" y2="10.16" width="0.4064" layer="1"/>
 <wire x1="28.448" y1="10.16" x2="28.448" y2="17.272" width="0.4064" layer="1"/>
 <wire x1="28.448" y1="17.272" x2="24.892" y2="20.828" width="0.4064" layer="1"/>
@@
 <wire x1="27.432" y1="50.8" x2="27.686" y2="50.8" width="0.4064" layer="16"/>
 </signal>
+<signal name="N$16">
+<contactref element="J4" pad="D12"/>
+<contactref element="J5" pad="2"/>
+<wire x1="34.036" y1="2.54" x2="34.036" y2="6.604" width="0.4064" layer="1"/>
+</signal>
+<signal name="N$17">
+<contactref element="J4" pad="D11"/>
+<contactref element="J5" pad="3"/>
+<wire x1="31.496" y1="2.54" x2="31.496" y2="6.604" width="0.4064" layer="1"/>
+</signal>
+<signal name="N$18">
+<contactref element="J4" pad="D10"/>
+<contactref element="J5" pad="4"/>
+<wire x1="28.956" y1="2.54" x2="28.956" y2="6.604" width="0.4064" layer="1"/>
+</signal>
+<signal name="N$19">
+<contactref element="J4" pad="D9"/>
+<contactref element="J5" pad="5"/>
+<wire x1="26.416" y1="2.54" x2="26.416" y2="6.604" width="0.4064" layer="1"/>
+</signal>
+<signal name="N$22">
+<contactref element="J4" pad="D8"/>
+<contactref element="J5" pad="6"/>
+<wire x1="23.876" y1="2.54" x2="23.876" y2="6.604" width="0.4064" layer="1"/>
+</signal>
+<signal name="N$23">
+<contactref element="J4" pad="D7"/>
+<contactref element="J5" pad="7"/>
+<wire x1="20.066" y1="2.54" x2="21.336" y2="3.81" width="0.4064" layer="1"/>
+<wire x1="21.336" y1="3.81" x2="21.336" y2="6.604" width="0.4064" layer="1"/>
+</signal>
+<signal name="N$24">
+<contactref element="J4" pad="D6"/>
+<contactref element="J5" pad="8"/>
+<wire x1="17.526" y1="2.54" x2="17.526" y2="3.81" width="0.4064" layer="1"/>
+<wire x1="17.526" y1="3.81" x2="18.796" y2="5.08" width="0.4064" layer="1"/>
+<wire x1="18.796" y1="5.08" x2="18.796" y2="6.604" width="0.4064" layer="1"/>
+</signal>
+<signal name="N$25">
+<contactref element="J4" pad="D5"/>
+<contactref element="J5" pad="9"/>
+<wire x1="14.986" y1="2.54" x2="14.986" y2="5.334" width="0.4064" layer="1"/>
+<wire x1="14.986" y1="5.334" x2="16.256" y2="6.604" width="0.4064" layer="1"/>
+</signal>
 </signals>
