File: boards/arduino-shield-xyz-stepper.sch (EAGLE design)
At the start: 8 parts, among them IC1 2967-MP6500, IC2 2967-MP6500, IC3 2967-MP6500, J4 ARDUINO_R3_SHIELD

Commit message: xyz stepper control
Parts:
- added J5: (no value), SparkFun-Connectors:CONN_09
Connections:
- new net N$16: J4.D12, J5.2
- new net N$17: J4.*D11, J5.3
- new net N$18: J4.*D10, J5.4
- new net N$19: J4.*D9, J5.5
- new net N$22: J4.D8, J5.6
- new net N$23: J4.D7, J5.7
- new net N$24: J4.*D6, J5.8
- new net N$25: J4.*D5, J5.9
- net GND: now also J5.1
Changed lines of the file:
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@@
 <part name="GND3" library="SparkFun-PowerSymbols" deviceset="GND" device=""/>
 <part name="SUPPLY7" library="SparkFun-PowerSymbols" deviceset="5V" device=""/>
+<part name="J5" library="SparkFun-Connectors" deviceset="CONN_09" device=""/>
+<part name="GND4" library="SparkFun-PowerSymbols" deviceset="GND" device=""/>
 </parts>
 <sheets>
@@
 </instance>
 <instance part="SUPPLY7" gate="G$1" x="45.72" y="100.33" rot="R90"/>
+<instance part="J5" gate="J1" x="102.87" y="97.79" rot="R180"/>
+<instance part="GND4" gate="1" x="107.95" y="121.92" smashed="yes">
+<attribute name="VALUE" x="107.95" y="121.666" size="1.778" layer="96" align="top-center"/>
+</instance>
 </instances>
 <busses>
@@
 <pinref part="GND3" gate="1" pin="GND"/>
 <wire x1="48.26" y1="110.49" x2="43.18" y2="110.49" width="0.1524" layer="91"/>
+</segment>
+<segment>
+<pinref part="J5" gate="J1" pin="1"/>
+<wire x1="92.71" y1="107.95" x2="86.36" y2="107.95" width="0.1524" layer="91"/>
+<wire x1="86.36" y1="107.95" x2="86.36" y2="124.46" width="0.1524" layer="91"/>
+<wire x1="86.36" y1="124.46" x2="107.95" y2="124.46" width="0.1524" layer="91"/>
+<pinref part="GND4" gate="1" pin="GND"/>
 </segment>
 </net>
@@
 </segment>
 </net>
+<net name="N$16" class="0">
+<segment>
+<pinref part="J4" gate="G$1" pin="D12"/>
+<pinref part="J5" gate="J1" pin="2"/>
+<wire x1="92.71" y1="105.41" x2="73.66" y2="105.41" width="0.1524" layer="91"/>
+</segment>
+</net>
+<net name="N$17" class="0">
+<segment>
+<pinref part="J4" gate="G$1" pin="*D11"/>
+<pinref part="J5" gate="J1" pin="3"/>
+<wire x1="92.71" y1="102.87" x2="73.66" y2="102.87" width="0.1524" layer="91"/>
+</segment>
+</net>
+<net name="N$18" class="0">
+<segment>
+<pinref part="J4" gate="G$1" pin="*D10"/>
+<pinref part="J5" gate="J1" pin="4"/>
+<wire x1="92.71" y1="100.33" x2="73.66" y2="100.33" width="0.1524" layer="91"/>
+</segment>
+</net>
+<net name="N$19" class="0">
+<segment>
+<pinref part="J4" gate="G$1" pin="*D9"/>
+<pinref part="J5" gate="J1" pin="5"/>
+<wire x1="92.71" y1="97.79" x2="73.66" y2="97.79" width="0.1524" layer="91"/>
+</segment>
+</net>
+<net name="N$22" class="0">
+<segment>
+<pinref part="J4" gate="G$1" pin="D8"/>
+<pinref part="J5" gate="J1" pin="6"/>
+<wire x1="92.71" y1="95.25" x2="73.66" y2="95.25" width="0.1524" layer="91"/>
+</segment>
+</net>
+<net name="N$23" class="0">
+<segment>
+<pinref part="J4" gate="G$1" pin="D7"/>
+<pinref part="J5" gate="J1" pin="7"/>
+<wire x1="92.71" y1="92.71" x2="73.66" y2="92.71" width="0.1524" layer="91"/>
+</segment>
+</net>
+<net name="N$24" class="0">
+<segment>
+<pinref part="J4" gate="G$1" pin="*D6"/>
+<pinref part="J5" gate="J1" pin="8"/>
+<wire x1="92.71" y1="90.17" x2="73.66" y2="90.17" width="0.1524" layer="91"/>
+</segment>
+</net>
+<net name="N$25" class="0">
+<segment>
+<pinref part="J4" gate="G$1" pin="*D5"/>
+<pinref part="J5" gate="J1" pin="9"/>
+<wire x1="92.71" y1="87.63" x2="73.66" y2="87.63" width="0.1524" layer="91"/>
+</segment>
+</net>
