File: boards/unoshield-v6.sch (EAGLE design)
At the start: 21 parts, among them J1 455-1750-1-ND, J4 ARDUINO_R3_SHIELD, SW1 BUTTON, SW2 BUTTON, SW3 ON-OFF-ON-360-1013-ND

Commit message: shield tweaks
Other:
- moved on the sheet: C1, D1, J1, J10, J11, J12, J2, J3, J5, J7, J8, J9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
