File: boards/unoshield-v6.brd (EAGLE design)
At the start: 54.6 x 63.5 mm, 21 parts, among them J1 455-1750-1-ND, J4 ARDUINO_R3_SHIELD, SW1 BUTTON, SW2 BUTTON, SW3 ON-OFF-ON-360-1013-ND

Commit message: shield tweaks
Routing:
- net N$6: track 78.8 -> 77.0 mm
Changed lines of the file:
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@@
 <contactref element="J10" pad="1"/>
 <wire x1="8.255" y1="62.23" x2="10.16" y2="62.23" width="0.6096" layer="16"/>
-<wire x1="10.16" y1="53.975" x2="16.51" y2="53.975" width="0.6096" layer="16"/>
-<wire x1="16.51" y1="53.975" x2="16.51" y2="49.824" width="0.6096" layer="16"/>
-<wire x1="15.073" y1="48.387" x2="16.51" y2="49.824" width="0.6096" layer="16"/>
+<wire x1="10.16" y1="53.975" x2="15.24" y2="53.975" width="0.6096" layer="16"/>
+<wire x1="15.24" y1="53.975" x2="15.24" y2="48.554" width="0.6096" layer="16"/>
+<wire x1="15.073" y1="48.387" x2="15.24" y2="48.554" width="0.6096" layer="16"/>
 <wire x1="10.16" y1="62.23" x2="10.16" y2="53.975" width="0.6096" layer="16"/>
 <wire x1="15.073" y1="48.387" x2="13.97" y2="47.284" width="0.6096" layer="1"/>

Commit message: gerbers zip made and submitted to pcbway
Parts:
- moved C1 1.40 mm to (14.0, 48.3)
- moved J12 1.27 mm to (30.5, 26.7)
- moved J6 1.27 mm to (35.6, 26.7)
- moved J9 1.27 mm to (40.6, 26.7)
Routing:
- net N$6: track 77.0 -> 60.4 mm
- net N$5: track 24.4 -> 23.1 mm
- net VIN: track 49.2 -> 50.4 mm
Changed lines of the file:
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@@
 <text x="39.37" y="59.182" size="1.016" layer="21" rot="R180">Button</text>
 <text x="36.576" y="20.32" size="1.016" layer="21" rot="R180">IRFL024NTRPBF</text>
-<text x="34.29" y="22.225" size="1.27" layer="21">Vin</text>
+<text x="34.29" y="23.495" size="1.27" layer="21">Vin</text>
 <text x="12.319" y="33.02" size="1.27" layer="21">5 V in</text>
 <text x="8.001" y="24.892" size="1.27" layer="21">GND</text>
-<text x="28.829" y="22.225" size="1.27" layer="21">5 V</text>
-<text x="38.989" y="22.225" size="1.27" layer="21">12 V</text>
+<text x="28.829" y="23.495" size="1.27" layer="21">5 V</text>
+<text x="38.989" y="23.495" size="1.27" layer="21">12 V</text>
 <text x="34.925" y="45.72" size="1.778" layer="21">10k</text>
 <wire x1="22.225" y1="8.255" x2="22.225" y2="5.715" width="0.6096" layer="21"/>
@@
 <elements>
 <element name="J4" library="SparkFun-Boards" package="UNO_R3_SHIELD" value="ARDUINO_R3_SHIELD" x="-0.508" y="-7.874" smashed="yes"/>
-<element name="C1" library="SparkFun-Capacitors" package="CPOL-RADIAL-1000UF-25V-KIT" value="1000uf/25V" x="12.573" y="48.387" smashed="yes">
-<attribute name="NAME" x="11.811" y="51.308" size="0.4064" layer="25"/>
-<attribute name="PROD_ID" value="CAP-09538" x="12.573" y="48.387" size="1.778" layer="27" display="off"/>
-<attribute name="VALUE" x="10.568" y="44.369" size="0.8128" layer="27"/>
+<element name="C1" library="SparkFun-Capacitors" package="CPOL-RADIAL-1000UF-25V-KIT" value="1000uf/25V" x="13.97" y="48.26" smashed="yes">
+<attribute name="NAME" x="13.208" y="51.181" size="0.4064" layer="25"/>
+<attribute name="PROD_ID" value="CAP-09538" x="13.97" y="48.26" size="1.778" layer="27" display="off"/>
+<attribute name="VALUE" x="11.965" y="44.242" size="0.8128" layer="27"/>
 </element>
 <element name="R5" library="SparkFun-Electromechanical" package="ALPS_POT_KIT" value="20k" x="29.591" y="43.688" smashed="yes" rot="R270"/>
@@
 <attribute name="VALUE" x="39.624" y="5.842" size="0.6096" layer="27" font="vector" ratio="20"/>
 </element>
-<element name="J6" library="SparkFun-Connectors" package="1X01" value="" x="35.56" y="25.4" smashed="yes">
-<attribute name="NAME" x="34.29" y="26.797" size="0.6096" layer="25" font="vector" ratio="20"/>
-<attribute name="VALUE" x="34.29" y="23.876" size="0.6096" layer="27" font="vector" ratio="20" align="top-left"/>
-</element>
-<element name="J9" library="SparkFun-Connectors" package="1X01" value="" x="40.64" y="25.4" smashed="yes">
-<attribute name="NAME" x="39.37" y="26.797" size="0.6096" layer="25" font="vector" ratio="20"/>
-<attribute name="VALUE" x="39.37" y="23.876" size="0.6096" layer="27" font="vector" ratio="20" align="top-left"/>
+<element name="J6" library="SparkFun-Connectors" package="1X01" value="" x="35.56" y="26.67" smashed="yes">
+<attribute name="NAME" x="34.29" y="28.067" size="0.6096" layer="25" font="vector" ratio="20"/>
+<attribute name="VALUE" x="34.29" y="25.146" size="0.6096" layer="27" font="vector" ratio="20" align="top-left"/>
+</element>
+<element name="J9" library="SparkFun-Connectors" package="1X01" value="" x="40.64" y="26.67" smashed="yes">
+<attribute name="NAME" x="39.37" y="28.067" size="0.6096" layer="25" font="vector" ratio="20"/>
+<attribute name="VALUE" x="39.37" y="25.146" size="0.6096" layer="27" font="vector" ratio="20" align="top-left"/>
 </element>
 <element name="J10" library="SparkFun-Connectors" package="1X01_2MM" value="" x="13.97" y="30.48" smashed="yes">
@@
 <attribute name="VALUE" x="12.319" y="22.987" size="0.6096" layer="27" font="vector" ratio="20"/>
 </element>
-<element name="J12" library="SparkFun-Connectors" package="1X01" value="" x="30.48" y="25.4" smashed="yes">
-<attribute name="NAME" x="29.21" y="26.797" size="0.6096" layer="25" font="vector" ratio="20"/>
-<attribute name="VALUE" x="29.21" y="23.876" size="0.6096" layer="27" font="vector" ratio="20" align="top-left"/>
+<element name="J12" library="SparkFun-Connectors" package="1X01" value="" x="30.48" y="26.67" smashed="yes">
+<attribute name="NAME" x="29.21" y="28.067" size="0.6096" layer="25" font="vector" ratio="20"/>
+<attribute name="VALUE" x="29.21" y="25.146" size="0.6096" layer="27" font="vector" ratio="20" align="top-left"/>
 </element>
 <element name="R7" library="SparkFun-Resistors" package="AXIAL-0.3" value="10k" x="19.685" y="10.16" smashed="yes" rot="R90">
@@
 <wire x1="35.179" y1="13.335" x2="35.179" y2="12.82" width="0.6096" layer="1"/>
 <wire x1="41.275" y1="13.335" x2="41.275" y2="15.875" width="0.6096" layer="16"/>
-<wire x1="40.64" y1="25.4" x2="40.64" y2="15.875" width="0.6096" layer="16"/>
+<wire x1="40.64" y1="26.67" x2="40.64" y2="15.875" width="0.6096" layer="16"/>
 <wire x1="13.97" y1="12.7" x2="13.97" y2="15.875" width="0.6096" layer="16"/>
 <wire x1="13.97" y1="15.875" x2="40.64" y2="15.875" width="0.6096" layer="16"/>
@@
 <wire x1="50.292" y1="28.956" x2="50.292" y2="31.75" width="0.6096" layer="1"/>
 <wire x1="50.292" y1="31.75" x2="35.56" y2="31.75" width="0.6096" layer="1"/>
-<wire x1="35.56" y1="31.75" x2="35.56" y2="25.4" width="0.6096" layer="1"/>
+<wire x1="35.56" y1="31.75" x2="35.56" y2="26.67" width="0.6096" layer="1"/>
 </signal>
 <signal name="N$6">
@@
 <contactref element="J10" pad="1"/>
 <wire x1="8.255" y1="62.23" x2="10.16" y2="62.23" width="0.6096" layer="16"/>
-<wire x1="10.16" y1="53.975" x2="15.24" y2="53.975" width="0.6096" layer="16"/>
-<wire x1="15.24" y1="53.975" x2="15.24" y2="48.554" width="0.6096" layer="16"/>
-<wire x1="15.073" y1="48.387" x2="15.24" y2="48.554" width="0.6096" layer="16"/>
-<wire x1="10.16" y1="62.23" x2="10.16" y2="53.975" width="0.6096" layer="16"/>
-<wire x1="15.073" y1="48.387" x2="13.97" y2="47.284" width="0.6096" layer="1"/>
-<wire x1="13.97" y1="30.48" x2="13.97" y2="47.284" width="0.6096" layer="1"/>
 <contactref element="J12" pad="1"/>
-<wire x1="14.1405" y1="46.1845" x2="13.97" y2="46.014" width="0.6096" layer="1"/>
-<wire x1="13.97" y1="30.48" x2="13.97" y2="46.1845" width="0.6096" layer="1"/>
-<wire x1="13.97" y1="46.1845" x2="14.1405" y2="46.1845" width="0.6096" layer="1"/>
-<wire x1="13.97" y1="30.48" x2="30.48" y2="30.48" width="0.6096" layer="1"/>
-<wire x1="30.48" y1="30.48" x2="30.48" y2="25.4" width="0.6096" layer="1"/>
+<wire x1="13.97" y1="30.48" x2="16.51" y2="30.48" width="0.6096" layer="1"/>
+<wire x1="16.51" y1="30.48" x2="30.48" y2="30.48" width="0.6096" layer="1"/>
+<wire x1="30.48" y1="30.48" x2="30.48" y2="26.67" width="0.6096" layer="1"/>
+<wire x1="10.16" y1="53.34" x2="16.51" y2="53.34" width="0.6096" layer="16"/>
+<wire x1="16.51" y1="53.34" x2="16.51" y2="48.26" width="0.6096" layer="16"/>
+<wire x1="16.51" y1="48.26" x2="16.47" y2="48.26" width="0.6096" layer="16"/>
+<wire x1="10.16" y1="62.23" x2="10.16" y2="53.34" width="0.6096" layer="16"/>
+<wire x1="16.47" y1="48.26" x2="16.51" y2="48.26" width="0.6096" layer="1"/>
+<wire x1="16.51" y1="48.26" x2="16.51" y2="30.48" width="0.6096" layer="1"/>
 </signal>
 </signals>
