File: boards/arduino-shield-xyz-slime-stepper-v1.sch (EAGLE design)
At the start: 26 parts, among them IC1 2967-MP6500, IC3 2967-MP6500, J4 ARDUINO_R3_SHIELD, J9 455-1750-1-ND

Commit message: two new boards, xyz and slime and xyzhbridge and slime
Parts:
- removed U$1: ADAFRUIT-TB6612, spietz-library-2:ADAFRUIT-TB6612
- added IC2: 2967-MP6500, pololu-stepper-driver:2967-MP6500
- added J5: (no value), SparkFun-Connectors:CONN_02
Connections:
- removed net AIN1: J4.*D11, U$1.AIN1
- removed net AIN2: J4.D12, U$1.AIN2
- removed net BIN1: J4.*D10, U$1.BIN1
- removed net BIN2: J4.*D9, U$1.BIN2
- removed net N$17: J1.3, U$1.MA2
- removed net PWMA: J4.D13, U$1.PWMA
- removed net PWMB: J4.D8, U$1.PWMB
- removed net STBY: U$1.STBY
- new net DIR3: IC2.DIR, J4.*D10
- new net EN3: IC2.!ENBL, J4.D8
- new net N$10: IC2.B2, J1.1
- new net STEP3: IC2.STEP, J4.*D9
- net 5V: now also IC2.!SLEEP, IC2.MS1, IC2.MS2; no longer U$1.VCC
- net GND: now also IC2.GND1, IC2.GND2; no longer U$1.G2, U$1.G3, U$1.GND
- net N$11: now also IC2.B1; no longer U$1.MB1
- net N$12: now also IC2.A1, J1.3; no longer J1.1, U$1.MB2
- net N$16: now also IC2.A2; no longer U$1.MA1
- net N$18: now also J5.2
- net VMOT3: now also IC2.VMOT; no longer U$1.VM
- net VTRANSISTOR: now also J5.1
Other:
- moved on the sheet: J1
